File: dist_board.sch (EAGLE design)
At the start: 34 parts, among them J1 2p-2.54, J10 2p-2.54, J11 2p-2.54, J12 2p-2.54, J13 2p-2.54, J14 2p-2.54, J15 2p-2.54, J16 2p-2.54, J17 2p-2.54, J18 2p-2.54, J19 4p-2.54, J2 2p-2.54, J20 4p-2.54, J21 4p-2.54, J22 4p-2.54, J3 2p-2.54, J4 2p-2.54, J5 2p-2.54, J6 2p-2.54, J7 2p-2.54, J8 2p-2.54, J9 2p-2.54, X1 BU-SMB-V, X10 BU-SMB-V, X11 BU-SMB-V, X12 BU-SMB-V, X2 BU-SMB-V, X3 BU-SMB-V, X4 BU-SMB-V, X5 BU-SMB-V, X6 BU-SMB-V, X7 BU-SMB-V, X8 BU-SMB-V, X9 BU-SMB-V

Commit message: ready for ordering 1
Parts:
- renumbered J13 to HV3, J14 to HV2, J15 to HV1, J16 to GROUND1, J17 to GROUND2, J18 to GROUND3, J22 to GROUND
Connections:
- net N$10: now also J10.1; no longer J9.1
- net N$11: now also J11.1; no longer J10.1
- net N$12: now also J12.1; no longer J11.1
- net N$13: now also J7.1; no longer J12.1
- net N$8: now also J8.1; no longer J7.1
- net N$9: now also J9.1; no longer J8.1
Other:
- moved on the sheet: J10, J11, J12, J7, J8, J9
