File: trig3_board.brd (EAGLE design)
At the start: 140 x 87 mm, 97 parts, among them J1 2p-2.54, J10 2p-2.54, J11 2p-2.54, J12 2p-2.54, J13 8pin, J14 2p-2.54, J15 2p-2.54, J16 2p-2.54, J17 2p-2.54, J18 8pin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

Commit message: VME board, ordered from JLCPCB
Parts:
- added J19: 6HE-160-VG64AC, 19inch:6HE_160-VG64AC
- moved 173OUT9 19.2 mm to (111.0, 51.0)
- moved OJ13 19.2 mm to (81.0, 50.1)
- moved OJ15 19.2 mm to (117.0, 40.0)
- moved 13X6 19.2 mm to (4.00, 44.0)
- moved 145OUT16 19.2 mm to (87.0, 30.1)
- moved 147OUT15 19.2 mm to (87.0, 20.1)
- moved 159OUT14 19.2 mm to (111.0, 20.0)
- moved 161OUT13 19.2 mm to (111.0, 30.0)
- moved 164OUT12 19.2 mm to (87.0, 51.1)
- moved 167OUT11 19.2 mm to (87.0, 41.1)
- moved 174OUT1 19.2 mm to (111.0, 93.0)
- moved 176OUT2 19.2 mm to (111.0, 83.0)
- moved 177OUT6 19.2 mm to (111.0, 62.0)
- moved 181OUT3 19.2 mm to (87.0, 83.1)
- moved 182OUT7 19.2 mm to (87.0, 62.1)
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Connections:
- net 5V: now also J19.1-A32, J19.1-C32, J19.2-A32, J19.2-C32
- net GND: now also J19.1-A9, J19.1-C9, J19.2-A9, J19.2-C9
Routing:
- net 5V: track 213.1 -> 433.0 mm
- net 186OE: track 181.5 -> 333.7 mm, vias 7 -> 0
- net IO49: track 44.6 -> 108.9 mm, vias 2 -> 0
- net IO39: track 58.7 -> 112.3 mm, vias 2 -> 0
- net IO147_IN3: track 73.0 -> 52.5 mm, vias 0 -> 2
- net IO236: track 38.0 -> 57.6 mm
- net IO43: track 86.3 -> 69.1 mm, vias 2 -> 0
- net IO164_IN4: track 43.2 -> 59.9 mm
- net GND: track 57.3 -> 45.4 mm, vias 2 -> 0
- net IO145_IN4: track 66.9 -> 56.6 mm, vias 0 -> 2
- net IO184_IN4: track 41.2 -> 49.9 mm, vias 0 -> 2
- net IO37: track 74.0 -> 82.0 mm
- net OUT6: track 23.1 -> 18.5 mm, vias 2 -> 0
- net OUT2: track 23.1 -> 18.5 mm, vias 2 -> 0
- net IO177_IN2: track 29.0 -> 33.3 mm
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- added copper zone on layer 1, net 5V
Other:
- board size 140 x 87 mm -> 233.2 x 160 mm
