File: trig4_board.sch (EAGLE design)
At the start: 99 parts, among them J1 2p-2.54, J10 2p-2.54, J11 2p-2.54, J12 2p-2.54, J13 8pin, J14 2p-2.54, J15 2p-2.54, J16 2p-2.54, J17 2p-2.54, J18 8pin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

Commit message: 4 layer
Connections:
- net IO185: now also J191-A30.MS, J192-A30.MS
- net IO187: now also J191-A29.MS, J192-A29.MS
- net IO189: now also J191-A28.MS, J192-A28.MS
- net IO195: now also J191-A27.MS, J192-A27.MS
Other:
- moved on the sheet: J192-A1, J192-A10, J192-A11, J192-A12, J192-A13, J192-A14, J192-A15, J192-A16, J192-A17, J192-A18, J192-A19, J192-A2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
