File: trig4_board.sch (EAGLE design)
At the start: 99 parts, among them J1 2p-2.54, J10 2p-2.54, J11 2p-2.54, J12 2p-2.54, J13 8pin, J14 2p-2.54, J15 2p-2.54, J16 2p-2.54, J17 2p-2.54, J18 8pin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

Commit message: add possibility of EP4CE10 board
Parts:
- added X1, X2: 87758-1616, con-molex:87758-1616
Other:
- note added: "For EP3C16 board"
- note added: "For EP4CE10 board"
- moved on the sheet: 13X6, 145OUT16, 147OUT15, 159OUT14, 161OUT13, 164OUT12, 167OUT11, 169OUT10, 173OUT9, 174OUT1, 175OUT5, 176OUT2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
