File: trig4_board.brd (EAGLE design)
At the start: 233.2 x 160 mm, 99 parts, among them J1 2p-2.54, J10 2p-2.54, J11 2p-2.54, J12 2p-2.54, J13 8pin, J14 2p-2.54, J15 2p-2.54, J16 2p-2.54, J17 2p-2.54, J18 8pin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

Commit message: 4 layer
Connections:
- net IO185: now also J19.1-A30, J19.2-A30
- net IO187: now also J19.1-A29, J19.2-A29
- net IO189: now also J19.1-A28, J19.2-A28
- net IO195: now also J19.1-A27, J19.2-A27
Routing:
- net IO195: track 18.4 -> 336.2 mm
- net IO185: track 16.8 -> 332.2 mm
- net IO187: track 17.9 -> 313.5 mm
- net IO189: track 19.0 -> 299.3 mm
- net 5V: track 275.9 -> 0.00 mm
- net 186OE: track 333.7 -> 157.8 mm, vias 0 -> 1
- net IO49: track 108.9 -> 43.7 mm
- net IO39: track 112.3 -> 57.3 mm
- net IO19: track 47.5 -> 86.0 mm, vias 1 -> 0
- net IO43: track 69.1 -> 50.1 mm
- net IO37: track 82.0 -> 63.3 mm
- net IO236: track 57.6 -> 38.9 mm
- net IO174_IN1: track 61.9 -> 44.5 mm, vias 0 -> 1
- net IO181_IN3: track 42.7 -> 58.6 mm, vias 3 -> 1
- net IO184_IN4: track 49.9 -> 39.8 mm, vias 2 -> 1
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- added copper zone on layer 15, net GND
- removed copper zone on layer 16, net GND
Other:
- board text added: "-12V"
- board text added: "12V"

Commit message: new routing
Parts:
- moved J20 18.4 mm to (58.0, -47.0), turned to 0 degrees
Connections:
- net -12V: no longer J19.2-A31
- net 12V: no longer J19.2-C31
- net 5V: no longer J19.2-A32, J19.2-C32
- net GND: no longer J19.2-A9, J19.2-C9
- net IO185: no longer J19.2-A30
- net IO187: no longer J19.2-A29
- net IO189: no longer J19.2-A28
- net IO195: no longer J19.2-A27
Routing:
- net IO195: track 336.2 -> 0.00 mm
- net IO185: track 332.2 -> 0.00 mm
- net IO187: track 313.5 -> 0.00 mm
- net IO189: track 299.3 -> 0.00 mm
- net -12V: track 141.7 -> 0.00 mm
- net 12V: track 141.5 -> 0.00 mm
- net IO19: track 86.0 -> 0.00 mm
- net IO21: track 70.7 -> 0.00 mm
- net IO37: track 63.3 -> 0.00 mm
- net IO39: track 57.3 -> 0.00 mm
- net IO159_IN2: track 59.3 -> 5.46 mm, vias 1 -> 0
- net IO147_IN3: track 58.7 -> 5.59 mm, vias 1 -> 0
- net IO181_IN3: track 58.6 -> 5.59 mm, vias 1 -> 0
- net 186OE: track 157.8 -> 105.4 mm, vias 1 -> 0
- net IO43: track 50.1 -> 0.00 mm
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Other:
- board text added: "--12V"
- board text removed: "-12V"

Commit message: add possibility of EP4CE10 board
Parts:
- added X1, X2: 87758-1616, con-molex:87758-1616
Other:
- board text added: "Waveshare CoreEP3C16 or CoreEP4CE10"
Changed lines of the file:
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@@
 <drawing>
 <settings>
-<setting alwaysvectorfont="no"/>
+<setting alwaysvectorfont="yes"/>
 <setting verticaltext="up"/>
 </settings>
-<grid distance="1" unitdist="mm" unit="mm" style="lines" multiple="1" display="no" altdistance="0.1" altunitdist="mm" altunit="mm"/>
+<grid distance="1" unitdist="mm" unit="mm" style="lines" multiple="1" display="yes" altdistance="0.1" altunitdist="mm" altunit="mm"/>
 <layers>
-<layer number="1" name="power" color="4" fill="1" visible="no" active="yes"/>
+<layer number="1" name="power" color="4" fill="1" visible="yes" active="yes"/>
 <layer number="2" name="route2" color="16" fill="1" visible="yes" active="yes"/>
 <layer number="3" name="Route3" color="4" fill="3" visible="no" active="no"/>
@@
 <text x="68.5" y="-42.4" size="0.8128" layer="21" rot="R270">5V</text>
 <text x="73.5" y="-42.4" size="0.8128" layer="21" rot="R270">5V</text>
+<wire x1="18" y1="88" x2="19" y2="88" width="0.1524" layer="21"/>
+<wire x1="19" y1="88" x2="75" y2="88" width="0.1524" layer="21"/>
+<wire x1="75" y1="88" x2="76" y2="87" width="0.1524" layer="21"/>
+<wire x1="76" y1="87" x2="76" y2="21" width="0.1524" layer="21"/>
+<wire x1="76" y1="21" x2="75" y2="20" width="0.1524" layer="21"/>
+<wire x1="75" y1="20" x2="18" y2="20" width="0.1524" layer="21"/>
+<wire x1="18" y1="20" x2="16" y2="22" width="0.1524" layer="21"/>
+<wire x1="16" y1="22" x2="16" y2="88" width="0.1524" layer="21"/>
+<wire x1="16" y1="88" x2="18" y2="88" width="0.1524" layer="21"/>
+<text x="32" y="52" size="1.778" layer="21">Waveshare
+CoreEP3C16
+or
+CoreEP4CE10</text>
 </plain>
 <attributes>
@@
 <attribute name="NAME" x="55.603" y="-47.27" size="0.8128" layer="25" font="vector" rot="R90"/>
 <attribute name="PROD_ID" value="CONN-08438" x="58" y="-47" size="1.778" layer="27" display="off"/>
+</element>
+<element name="X1" library="con-molex" library_urn="urn:adsk.eagle:library:165" package="87758-1616" value="87758-1616" x="39" y="25">
+<attribute name="MF" value="MOLEX" x="39" y="25" size="1.778" layer="27" display="off"/>
+<attribute name="MPN" value="87758-1616" x="39" y="25" size="1.778" layer="27" display="off"/>
+<attribute name="NAME" x="31.38" y="21.19" size="1.27" layer="25"/>
+<attribute name="OC_FARNELL" value="7472366" x="39" y="25" size="1.778" layer="27" display="off"/>
+<attribute name="OC_NEWARK" value="59J1563" x="39" y="25" size="1.778" layer="27" display="off"/>
+</element>
+<element name="X2" library="con-molex" library_urn="urn:adsk.eagle:library:165" package="87758-1616" value="87758-1616" x="55" y="25">
+<attribute name="MF" value="MOLEX" x="55" y="25" size="1.778" layer="27" display="off"/>
+<attribute name="MPN" value="87758-1616" x="55" y="25" size="1.778" layer="27" display="off"/>
+<attribute name="NAME" x="47.38" y="21.19" size="1.27" layer="25"/>
+<attribute name="OC_FARNELL" value="7472366" x="55" y="25" size="1.778" layer="27" display="off"/>
+<attribute name="OC_NEWARK" value="59J1563" x="55" y="25" size="1.778" layer="27" display="off"/>
 </element>
 </elements>
@@
 </drawing>
 <compatibility>
+<note version="6.3" minversion="6.2.2" severity="warning">
+Since Version 6.2.2 text objects can contain more than one line,
+which will not be processed correctly with this version.
+</note>
 <note version="8.2" severity="warning">
 Since Version 8.2, EAGLE supports online libraries. The ids
