File: haasoscope_triggerout_board.sch (EAGLE design)
At the start: 6 parts, among them J1 2p-2.54, J2 2p-2.54

Commit message: trigout board
Parts:
- added J3, J4: 2p-2.54, Seeed-Connector:DIP-BLACK-MALE-HEADER-VERT(2P-2.54)
- added O10, O8: BU-SMB-V, con-coax:BU-SMB-V
Connections:
- net A10: now also J4.2, O10.1
- net A8: now also J3.2, O8.1
- net GND: now also J3.1, J4.1, O10.2, O8.2
Other:
- moved on the sheet: JP1, JP2
