File: trig3_board_trigger_waveshare_lvds.brd (EAGLE design)
At the start: 233.2 x 160 mm, 86 parts, among them IC1 SN65LVDT388ADBT, IC2 SN65LVDT388ADBT, IC3 SN65LVDT388ADBT, IC4 SN65LVDT388ADBT, IC5 SN65LVDT388ADBT, IC6 SN65LVDT388ADBT, IC7 SN65LVDT388ADBT, IC8 SN65LVDT388ADBT, J12 4p-2.54, J19 6HE-160-VG64AC, J20 8pin, J3 4p-2.54, J4 4p-2.54, X1 87758-1616, X13 87758-2816, X14 87758-2816, X15 87758-1616, X16 87758-1616, X17 87758-2816, X18 87758-2816, X2 87758-1616

Commit message: routed
Parts:
- moved CP11 101.0 mm to (166.0, -31.0)
- moved CP2 101.0 mm to (166.0, -26.0)
- moved CP6 101.0 mm to (167.0, -20.0)
- moved REG 101.0 mm to (158.0, -23.0)
- moved LEDPOW 71.0 mm to (148.0, -20.0)
- moved RLEDPOW 71.0 mm to (148.0, -26.0)
- moved LED1 19.4 mm to (173.0, 86.0)
- moved R8 19.4 mm to (173.0, 80.0)
- moved J12 12.0 mm to (145.0, 104.0)
- moved J4 12.0 mm to (157.0, 104.0)
- moved R1 4.00 mm to (173.0, 93.0)
Routing:
- net 3V3: track 0.00 -> 675.9 mm
- net GND: track 0.00 -> 489.8 mm, vias 0 -> 17
- net 5V: track 0.00 -> 460.3 mm, vias 0 -> 2
- net OE: track 0.00 -> 318.2 mm, vias 0 -> 1
- net IN62: track 0.00 -> 157.8 mm, vias 0 -> 2
- net IN63: track 0.00 -> 157.5 mm, vias 0 -> 1
- net IN64: track 0.00 -> 145.7 mm, vias 0 -> 1
- net IN61: track 0.00 -> 142.5 mm, vias 0 -> 1
- net IO7: track 0.00 -> 139.2 mm
- net IO5: track 0.00 -> 134.9 mm, vias 0 -> 1
- net IO6: track 0.00 -> 126.4 mm, vias 0 -> 1
- net IN60: track 0.00 -> 125.5 mm, vias 0 -> 2
- net IN59: track 0.00 -> 123.8 mm, vias 0 -> 2
- net IN58: track 0.00 -> 120.0 mm, vias 0 -> 2
- net IN57: track 0.00 -> 117.0 mm, vias 0 -> 2
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- added copper zone on layer 16, net GND
- added copper zone on layer 2, net GND
- removed copper zone on layer 1, net GND
- removed copper zone on layer 15, net GND
Other:
- board text added: "3V3"
- board text added: "IO1"
- board text added: "IO2"
- board text added: "IO3"
- board text added: "IO4"
- board text added: "IO5"
- board text added: "IO6"
- board text added: "IO7"
- board text added: "OE"

Commit message: better
Parts:
- added IN65, IN66, IN67, IN68, IN69, IN70, IN71, IN72, IN73, IN74, IN75, IN76, IN77, IN78, IN79, IN80, OUT17, OUT18, OUT19, OUT20, OUT21, OUT22, OUT23, OUT24, OUT25, OUT26, OUT27, OUT28, OUT29, OUT30, OUT31, OUT32: BU-SMB-V, con-coax:BU-SMB-V
- added J1, J10, J11, J13, J14, J15, J16, J17, J2, J5, J6, J7, J8, J9: 8pin, SparkFun-Connectors:1X08
- LED_OE: value Red -> OutputEn
- moved CP11 113.0 mm to (164.0, 82.0)
- moved CP2 113.0 mm to (164.0, 87.0)
- moved CP6 113.0 mm to (165.0, 93.0)
- moved LEDPOW 113.0 mm to (146.0, 93.0)
- moved REG 113.0 mm to (156.0, 90.0)
- moved RLEDPOW 113.0 mm to (146.0, 87.0)
- moved C10 6.08 mm to (54.0, 88.0)
- moved C11 6.08 mm to (120.0, 88.0)
- moved C12 6.08 mm to (98.0, 88.0)
- moved C5 6.08 mm to (-34.0, 88.0)
- moved C6 6.08 mm to (-12.0, 88.0)
- moved C7 6.08 mm to (32.0, 88.0)
- moved C8 6.08 mm to (10.0, 88.0)
- moved C9 6.08 mm to (76.0, 88.0)
- renumbered 145OUT16 to OUT16, 147OUT15 to OUT15, 159OUT14 to OUT14, 161OUT13 to OUT13, 164OUT12 to OUT12, 167OUT11 to OUT11, 169OUT10 to OUT10, 173OUT9 to OUT9, 174OUT1 to OUT1, 175OUT5 to OUT5, 176OUT2 to OUT2, 177OUT6 to OUT6, 181OUT3 to OUT3, 182OUT7 to OUT7, 183OUT4 to OUT4, 184OUT8 to OUT8, LED1 to LED_OE
Connections:
- removed net IO145_IN4: VSLUE4.15, VSLUE4.17, X13.28
- removed net IO147_IN3: VSLUE4.11, VSLUE4.13, X13.26
- removed net IO159_IN2: VSLUE4.6, VSLUE4.8, X13.22
- removed net IO161_IN1: VSLUE4.2, VSLUE4.4, X13.20
- removed net IO164_IN4: VSLUE3.15, VSLUE3.17, X13.18
- removed net IO167_IN3: VSLUE3.11, VSLUE3.13, X13.16
- removed net IO169_IN2: VSLUE3.6, VSLUE3.8, X13.14
- removed net IO173_IN1: VSLUE3.2, VSLUE3.4, X13.12
- removed net IO174_IN1: VSLUE.2, VSLUE.4, X13.9
- removed net IO175_IN1: VSLUE2.2, VSLUE2.4, X13.10
- removed net IO176_IN2: VSLUE.6, VSLUE.8, X13.7
- removed net IO177_IN2: VSLUE2.6, VSLUE2.8, X13.8
- removed net IO181_IN3: VSLUE.11, VSLUE.13, X13.5
- removed net IO182_IN3: VSLUE2.11, VSLUE2.13, X13.6
- removed net IO183_IN4: VSLUE.15, VSLUE.17, X13.3
- removed net IO184_IN4: VSLUE2.15, VSLUE2.17, X13.4
- removed net N$130: X17.25
- removed net N$155: X17.26
- removed net N$182: X14.25
- removed net N$183: X14.23
- removed net N$184: X14.21
- removed net N$185: X14.19
- removed net N$186: X14.17
- removed net N$187: X14.15
- removed net N$188: X14.13
- removed net N$189: X14.11
- removed net N$190: X14.9
- removed net N$191: X14.7
- removed net N$192: X14.5
- removed net N$193: X14.3
- removed net N$194: X14.1
- removed net N$195: X14.26
- removed net N$196: X14.24
- removed net N$197: X14.22
- removed net N$198: X14.20
- removed net N$199: X14.18
- removed net N$200: X14.16
- removed net N$201: X14.14
- removed net N$202: X14.12
- removed net N$203: X14.10
- removed net N$204: X14.8
- removed net N$205: X14.6
- removed net N$206: X14.4
- removed net N$207: X14.2
- removed net N$217: X16.1
- removed net N$218: X16.3
- removed net N$219: X16.5
- removed net N$220: X16.7
- removed net N$221: X16.9
- removed net N$222: X16.11
- removed net N$223: X16.13
- removed net N$224: X16.15
- removed net N$225: X15.1
- removed net N$226: X15.3
- removed net N$227: X15.5
- removed net N$228: X15.7
- removed net N$229: X15.9
- removed net N$230: X15.11
- removed net N$231: X15.13
- removed net N$232: X15.15
- removed net N$249: X1.2
- removed net N$250: X1.4
- removed net N$251: X1.6
- removed net N$252: X1.8
- new net IN65: IN65.1, J7.8, X16.1
- new net IN66: IN66.1, J7.7, X16.3
- new net IN67: IN67.1, J7.6, X16.5
- new net IN68: IN68.1, J7.5, X16.7
- new net IN69: IN69.1, J7.4, X16.9
- new net IN70: IN70.1, J7.3, X16.11
- new net IN71: IN71.1, J7.2, X16.13
- new net IN72: IN72.1, J7.1, X16.15
- new net IN73: IN73.1, J8.8, X15.1
- new net IN74: IN74.1, J8.7, X15.3
- new net IN75: IN75.1, J8.6, X15.5
- new net IN76: IN76.1, J8.5, X15.7
- new net IN77: IN77.1, J8.4, X15.9
- new net IN78: IN78.1, J8.3, X15.11
- new net IN79: IN79.1, J8.2, X15.13
- new net IN80: IN80.1, J8.1, X15.15
- new net IO10: J14.6, X14.5
- new net IO11: J14.5, X14.7
- new net IO12: J14.4, X14.9
- new net IO13: J14.3, X14.11
- new net IO14: J14.2, X14.13
- new net IO15: J14.1, X14.15
- new net IO16: J15.8, X14.2
- new net IO17: J15.7, X14.4
- new net IO18: J15.6, X14.6
- new net IO19: J15.5, X14.8
- new net IO20: J15.4, X14.10
- new net IO21: J15.3, X14.12
- new net IO22: J15.2, X14.14
- new net IO23: J15.1, X14.16
- new net IO8: J14.8, X14.1
- new net IO9: J14.7, X14.3
- new net OUT10IN: J2.4, VSLUE3.6, VSLUE3.8, X13.14
- new net OUT11IN: J2.6, VSLUE3.11, VSLUE3.13, X13.16
- new net OUT12IN: J2.8, VSLUE3.15, VSLUE3.17, X13.18
- new net OUT13IN: J5.2, VSLUE4.2, VSLUE4.4, X13.20
- new net OUT14IN: J5.4, VSLUE4.6, VSLUE4.8, X13.22
- new net OUT15IN: J5.6, VSLUE4.11, VSLUE4.13, X13.26
- new net OUT16IN: J5.8, VSLUE4.15, VSLUE4.17, X13.28
- new net OUT17: J17.1, OUT17.1, X17.25
- new net OUT18: J17.2, OUT18.1, X17.26
- new net OUT19: J17.3, OUT19.1, X14.17
- new net OUT1IN: J1.2, VSLUE.2, VSLUE.4, X13.9
- new net OUT20: J17.4, OUT20.1, X14.19
- new net OUT21: J17.5, OUT21.1, X14.21
- new net OUT22: J17.6, OUT22.1, X14.23
- new net OUT23: J17.7, OUT23.1, X14.25
- new net OUT24: J17.8, OUT24.1, X14.18
- new net OUT25: J16.1, OUT25.1, X14.20
- new net OUT26: J16.2, OUT26.1, X14.22
- new net OUT27: J16.3, OUT27.1, X14.24
- new net OUT28: J16.4, OUT28.1, X14.26
- new net OUT29: J16.5, J9.8, OUT29.1, X1.2, X17.27
- new net OUT2IN: J1.4, VSLUE.6, VSLUE.8, X13.7
- new net OUT30: J16.6, J9.7, OUT30.1, X1.4, X17.28
- new net OUT31: J16.7, J9.6, OUT31.1, X1.6, X14.27
- new net OUT32: J16.8, J9.5, OUT32.1, X1.8, X14.28
- new net OUT3IN: J1.6, VSLUE.11, VSLUE.13, X13.5
- new net OUT4IN: J1.8, VSLUE.15, VSLUE.17, X13.3
- new net OUT5IN: J6.2, VSLUE2.2, VSLUE2.4, X13.10
- new net OUT6IN: J6.4, VSLUE2.6, VSLUE2.8, X13.8
- new net OUT7IN: J6.6, VSLUE2.11, VSLUE2.13, X13.6
- new net OUT8IN: J6.8, VSLUE2.15, VSLUE2.17, X13.4
- new net OUT9IN: J2.2, VSLUE3.2, VSLUE3.4, X13.12
- net GND: now also IN65.2, IN65.3, IN65.4, IN65.5, IN66.2, IN66.3, IN66.4, IN66.5, IN67.2, IN67.3, IN67.4, IN67.5, IN68.2, IN68.3, IN68.4, IN68.5, IN69.2, IN69.3, IN69.4, IN69.5, IN70.2, IN70.3, IN70.4, IN70.5, IN71.2, IN71.3, IN71.4, IN71.5, IN72.2, IN72.3, IN72.4, IN72.5, IN73.2, IN73.3, IN73.4, IN73.5, IN74.2, IN74.3, IN74.4, IN74.5, IN75.2, IN75.3, IN75.4, IN75.5, IN76.2, IN76.3, IN76.4, IN76.5, IN77.2, IN77.3, IN77.4, IN77.5, IN78.2, IN78.3, IN78.4, IN78.5, IN79.2, IN79.3, IN79.4, IN79.5, IN80.2, IN80.3, IN80.4, IN80.5, J1.1, J1.3, J1.5, J1.7, J2.1, J2.3, J2.5, J2.7, J5.1, J5.3, J5.5, J5.7, J6.1, J6.3, J6.5, J6.7, OUT17.2, OUT17.3, OUT17.4, OUT17.5, OUT18.2, OUT18.3, OUT18.4, OUT18.5, OUT19.2, OUT19.3, OUT19.4, OUT19.5, OUT20.2, OUT20.3, OUT20.4, OUT20.5, OUT21.2, OUT21.3, OUT21.4, OUT21.5, OUT22.2, OUT22.3, OUT22.4, OUT22.5, OUT23.2, OUT23.3, OUT23.4, OUT23.5, OUT24.2, OUT24.3, OUT24.4, OUT24.5, OUT25.2, OUT25.3, OUT25.4, OUT25.5, OUT26.2, OUT26.3, OUT26.4, OUT26.5, OUT27.2, OUT27.3, OUT27.4, OUT27.5, OUT28.2, OUT28.3, OUT28.4, OUT28.5, OUT29.2, OUT29.3, OUT29.4, OUT29.5, OUT30.2, OUT30.3, OUT30.4, OUT30.5, OUT31.2, OUT31.3, OUT31.4, OUT31.5, OUT32.2, OUT32.3, OUT32.4, OUT32.5
- net N$253: now also J9.4
- net N$254: now also J9.3
- net N$255: now also J9.2
- net N$256: now also J9.1
- net N$257: now also J10.8
- net N$258: now also J10.7
- net N$259: now also J10.6
- net N$260: now also J10.5
- net N$261: now also J10.4
- net N$262: now also J10.3
- net N$263: now also J10.2
- net N$264: now also J10.1
- net N$265: now also J11.8
- net N$266: now also J11.7
- net N$267: now also J11.6
- net N$268: now also J11.5
- net N$269: now also J11.4
- net N$270: now also J11.3
- net N$271: now also J11.2
- net N$272: now also J11.1
- net N$273: now also J13.8
- net N$274: now also J13.7
- net N$275: now also J13.6
- net N$276: now also J13.5
- net N$277: now also J13.4
- net N$278: now also J13.3
- net N$279: now also J13.2
- net N$280: now also J13.1
Routing:
- net OUT19: track 0.00 -> 179.3 mm
- net OUT20: track 0.00 -> 165.0 mm
- net IN74: track 0.00 -> 157.0 mm, vias 0 -> 1
- net OUT21: track 0.00 -> 152.6 mm
- net OUT17: track 0.00 -> 147.7 mm
- net OUT18: track 0.00 -> 138.2 mm
- net OUT9IN: track 0.00 -> 125.6 mm, vias 0 -> 2
- net OUT14IN: track 0.00 -> 125.0 mm, vias 0 -> 1
- net 3V3: track 675.9 -> 552.6 mm
- net OUT15IN: track 0.00 -> 121.7 mm, vias 0 -> 1
- net OUT8IN: track 0.00 -> 120.1 mm, vias 0 -> 2
- net OUT29: track 0.00 -> 118.9 mm
- net OUT16IN: track 0.00 -> 117.4 mm, vias 0 -> 1
- net IN73: track 0.00 -> 116.3 mm, vias 0 -> 3
- net OUT23: track 0.00 -> 115.4 mm
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Other:
- board text added: "-12V"
- board text added: "EP4CE10 only"
- board text added: "IN65"
- board text added: "IN72"
- board text added: "IN73"
- board text added: "IN80"
- board text added: "IO15"
- board text added: "IO16"
- board text added: "IO23"
- board text added: "IO8"
- board text added: "OU12IN"
- board text added: "OUT10IN"
- board text added: "OUT11IN"
- board text added: "OUT13IN"
- board text added: "OUT14IN"
- board text added: "OUT15IN"
- board text added: "OUT16IN"
- board text added: "OUT17"
- board text added: "OUT1IN"
- board text added: "OUT24"
- board text added: "OUT25"
- board text added: "OUT29"
- board text added: "OUT2IN"
- board text added: "OUT32"
- board text added: "OUT3IN"
- board text added: "OUT4IN"
- board text added: "OUT5IN"
- board text added: "OUT6IN"
- board text added: "OUT7IN"
- board text added: "OUT8IN"
- board text added: "OUT9IN"
- board text removed: "--12V"
