File: trig3_board_de0-nano_extender/trig3_board_de0-nano_rack.brd (EAGLE design)
At the start: 276 x 100 mm, 274 parts, among them J10 2p-2.54, J11 2p-2.54, J12 4p-2.54, J13 BU-SMB-V, J131 4p-2.54, J14 BU-SMB-V, J141 2p-2.54, J15 2p-2.54, J16 2p-2.54, J17 2p-2.54, J18 2p-2.54, J22 2p-2.54, J23 2p-2.54, J24 2p-2.54, J25 2p-2.54, J28 2p-2.54, J29 2p-2.54, J3 4p-2.54, J30 2p-2.54, J31 2p-2.54, J311 4p-2.54, J32 2p-2.54, J33 2p-2.54, J34 2p-2.54, J35 2p-2.54, J36 2p-2.54, J37 2p-2.54, J38 2p-2.54, J39 2p-2.54, J4 2p-2.54, J40 2p-2.54, J41 2p-2.54, J42 2p-2.54, J43 2p-2.54, J48 2p-2.54, J49 2p-2.54, J5 2p-2.54, J50 2p-2.54, J51 2p-2.54, J52 2p-2.54, J53 2p-2.54, J54 2p-2.54, J55 2p-2.54, J6 2p-2.54, J7 4p-2.54, J8 2p-2.54, J9 2p-2.54, K15_R10P BU-SMB-V, K16_R10N BU-SMB-V, M16CLK_3N BU-SMB-V, P11 BU-SMB-V, P14_CLKOUT_4P BU-SMB-V, P15 BU-SMB-V, P16_R15N BU-SMB-V, P9 BU-SMB-V, T10_B16N BU-SMB-V, T12_B18N BU-SMB-V, T13_B20N BU-SMB-V, T14_B23P_SPARE BU-SMB-V, T15_B23N_TRIGOUT BU-SMB-V, T9CLK_7N BU-SMB-V

Commit message: add 6mm on top and bottom, to fit in sliders
Other:
- board size 276 x 100 mm -> 276 x 112 mm
Changed lines of the file:
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@@
 <setting verticaltext="up"/>
 </settings>
-<grid distance="2.54" unitdist="mm" unit="mm" style="lines" multiple="1" display="no" altdistance="0.1" altunitdist="mm" altunit="mm"/>
+<grid distance="1" unitdist="mm" unit="mm" style="lines" multiple="1" display="yes" altdistance="0.1" altunitdist="mm" altunit="mm"/>
 <layers>
 <layer number="1" name="Top" color="4" fill="1" visible="yes" active="yes"/>
@@
 <text x="103" y="-42" size="1.778" layer="21" rot="R180">de0-nano_2x13 board</text>
 <text x="87" y="34" size="1.27" layer="21">N9 (Outputs Enabled)</text>
-<wire x1="-45" y1="-63" x2="-45" y2="37" width="0.1524" layer="20"/>
-<wire x1="-45" y1="37" x2="231" y2="37" width="0.1524" layer="20"/>
-<wire x1="231" y1="37" x2="231" y2="-63" width="0.1524" layer="20"/>
-<wire x1="231" y1="-63" x2="-45" y2="-63" width="0.1524" layer="20"/>
-<dimension x1="-33" y1="-63" x2="-33" y2="37" x3="-47" y3="-13" textsize="1.778" layer="20" visible="yes"/>
-<dimension x1="231" y1="-68" x2="-45" y2="-68" x3="93" y3="-65.877821875" textsize="1.778" layer="20" visible="yes"/>
-<dimension x1="115" y1="-68" x2="-45" y2="-68" x3="35" y3="-69" textsize="1.778" layer="20"/>
-<dimension x1="-46" y1="-63" x2="-46" y2="-22" x3="-45" y3="-42.5" textsize="1.778" layer="20" visible="yes"/>
+<wire x1="-45" y1="-69" x2="-45" y2="43" width="0.1524" layer="20"/>
+<wire x1="-45" y1="43" x2="231" y2="43" width="0.1524" layer="20"/>
+<wire x1="231" y1="43" x2="231" y2="-69" width="0.1524" layer="20"/>
+<wire x1="231" y1="-69" x2="-45" y2="-69" width="0.1524" layer="20"/>
+<dimension x1="-33" y1="-63" x2="-33" y2="37" x3="-47" y3="-13" textsize="1.778" layer="21" visible="yes"/>
+<dimension x1="231" y1="-68" x2="-45" y2="-68" x3="93" y3="-65.877821875" textsize="1.778" layer="21" visible="yes"/>
+<dimension x1="115" y1="-68" x2="-45" y2="-68" x3="35" y3="-69" textsize="1.778" layer="21"/>
+<dimension x1="-46" y1="-63" x2="-46" y2="-22" x3="-45" y3="-42.5" textsize="1.778" layer="21" visible="yes"/>
 </plain>
 <attributes>
