File: trig3_board_de0-nano_extender/trig3_board_de0-nano_rack.brd (EAGLE design)
At the start: 276 x 112 mm, 274 parts, among them J10 2p-2.54, J11 2p-2.54, J12 4p-2.54, J13 BU-SMB-V, J131 4p-2.54, J14 BU-SMB-V, J141 2p-2.54, J15 2p-2.54, J16 2p-2.54, J17 2p-2.54, J18 2p-2.54, J22 2p-2.54, J23 2p-2.54, J24 2p-2.54, J25 2p-2.54, J28 2p-2.54, J29 2p-2.54, J3 4p-2.54, J30 2p-2.54, J31 2p-2.54, J311 4p-2.54, J32 2p-2.54, J33 2p-2.54, J34 2p-2.54, J35 2p-2.54, J36 2p-2.54, J37 2p-2.54, J38 2p-2.54, J39 2p-2.54, J4 2p-2.54, J40 2p-2.54, J41 2p-2.54, J42 2p-2.54, J43 2p-2.54, J48 2p-2.54, J49 2p-2.54, J5 2p-2.54, J50 2p-2.54, J51 2p-2.54, J52 2p-2.54, J53 2p-2.54, J54 2p-2.54, J55 2p-2.54, J6 2p-2.54, J7 4p-2.54, J8 2p-2.54, J9 2p-2.54, K15_R10P BU-SMB-V, K16_R10N BU-SMB-V, M16CLK_3N BU-SMB-V, P11 BU-SMB-V, P14_CLKOUT_4P BU-SMB-V, P15 BU-SMB-V, P16_R15N BU-SMB-V, P9 BU-SMB-V, T10_B16N BU-SMB-V, T12_B18N BU-SMB-V, T13_B20N BU-SMB-V, T14_B23P_SPARE BU-SMB-V, T15_B23N_TRIGOUT BU-SMB-V, T9CLK_7N BU-SMB-V

Commit message: routed with gnd on layers 2 and 15
Connections:
- net N$9 renamed LED1R
Routing:
- net 5V: track 26.6 -> 601.6 mm, vias 12 -> 0
- net GPIO_114_N9: track 541.0 -> 691.5 mm, vias 13 -> 5
- net GPIO_07_B5: track 139.3 -> 226.7 mm, vias 2 -> 3
- net GPIO_03_A3: track 277.2 -> 196.9 mm, vias 0 -> 2
- net GPIO_04_B3: track 153.4 -> 214.1 mm, vias 3 -> 2
- net GPIO_017_E6: track 133.3 -> 188.7 mm, vias 4 -> 1
- net GPIO_024_C9: track 209.0 -> 254.5 mm, vias 3 -> 1
- net GPIO_211_G16: track 166.1 -> 210.2 mm, vias 2 -> 0
- net GPIO_118_R16: track 171.1 -> 213.2 mm, vias 2 -> 1
- net GPIO_126_L14: track 113.7 -> 155.5 mm, vias 1 -> 2
- net GPIO_1_IN1_R9CLK_CLKIN: track 150.9 -> 190.8 mm, vias 4 -> 1
- net 3V3: track 201.2 -> 238.5 mm
- net GPIO_028_C11: track 86.8 -> 118.4 mm, vias 4 -> 2
- net GPIO_21_B16: track 172.3 -> 203.2 mm, vias 3 -> 1
- net GPIO_128_M10: track 113.6 -> 144.2 mm, vias 1 -> 0
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- added copper zone on layer 15, net GND
- removed copper zone on layer 15, net 5V
