File: trig3_board_de0-nano_extender/trig3_board_de0-nano_rack.sch (EAGLE design)
At the start: 274 parts, among them J10 2p-2.54, J11 2p-2.54, J12 4p-2.54, J13 BU-SMB-V, J131 4p-2.54, J14 BU-SMB-V, J141 2p-2.54, J15 2p-2.54, J16 2p-2.54, J17 2p-2.54, J18 2p-2.54, J22 2p-2.54, J23 2p-2.54, J24 2p-2.54, J25 2p-2.54, J28 2p-2.54, J29 2p-2.54, J3 4p-2.54, J30 2p-2.54, J31 2p-2.54, J311 4p-2.54, J32 2p-2.54, J33 2p-2.54, J34 2p-2.54, J35 2p-2.54, J36 2p-2.54, J37 2p-2.54, J38 2p-2.54, J39 2p-2.54, J4 2p-2.54, J40 2p-2.54, J41 2p-2.54, J42 2p-2.54, J43 2p-2.54, J48 2p-2.54, J49 2p-2.54, J5 2p-2.54, J50 2p-2.54, J51 2p-2.54, J52 2p-2.54, J53 2p-2.54, J54 2p-2.54, J55 2p-2.54, J6 2p-2.54, J7 4p-2.54, J8 2p-2.54, J9 2p-2.54, K15_R10P BU-SMB-V, K16_R10N BU-SMB-V, M16CLK_3N BU-SMB-V, P11 BU-SMB-V, P14_CLKOUT_4P BU-SMB-V, P15 BU-SMB-V, P16_R15N BU-SMB-V, P9 BU-SMB-V, T10_B16N BU-SMB-V, T12_B18N BU-SMB-V, T13_B20N BU-SMB-V, T14_B23P_SPARE BU-SMB-V, T15_B23N_TRIGOUT BU-SMB-V, T9CLK_7N BU-SMB-V

Commit message: routed with gnd on layers 2 and 15
Connections:
- net N$9 renamed LED1R
Changed lines of the file:
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@@
 </segment>
 </net>
-<net name="5V" class="3">
+<net name="5V" class="1">
 <segment>
 <pinref part="VSLUE" gate="G$1" pin="VCC"/>
@@
 </segment>
 </net>
-<net name="3V3" class="0">
+<net name="3V3" class="1">
 <segment>
 <pinref part="SV1" gate="G$1" pin="29"/>
@@
 </segment>
 </net>
-<net name="N$9" class="0">
+<net name="LED1R" class="1">
 <segment>
 <pinref part="LED1" gate="G$1" pin="C"/>
