File: trig3_board_de0-nano_extender/trig3_board_de0-nano_lvds.sch (EAGLE design)
At the start: 105 parts, among them IC1 SN65LVDT388ADBT, IC2 SN65LVDT388ADBT, IC3 SN65LVDT388ADBT, IC4 SN65LVDT388ADBT, IC5 SN65LVDT388ADBT, IC6 SN65LVDT388ADBT, IC7 SN65LVDT388ADBT, IC8 SN65LVDT388ADBT, J1 16, J12 4p-2.54, J131 4p-2.54, J14 BU-SMB-V, J19 6HE-160-VG64AC, J2 16, J3 4p-2.54, J311 4p-2.54, J4 4p-2.54

Commit message: try rj45 jack
Parts:
- removed JP1: 16, pinhead:PINHD-2X8/90
- added J5, J6: RJ45, SparkFun-Connectors:RJ45-8PTH
Connections:
- removed net N$19: IC1.D2A, JP1.15
- removed net N$20: IC1.D2B, JP1.16
- new net N$1: IC1.A1A, J5.8
- new net N$3: IC1.A2A, J5.6
- net N$10: now also IC1.B2B, J5.1; no longer IC1.B1B, JP1.6
- net N$11: now also IC1.C1A, J6.8; no longer IC1.B2A, JP1.7
- net N$12: now also IC1.C1B, J6.7; no longer IC1.B2B, JP1.8
- net N$13: now also IC1.C2A, J6.6; no longer IC1.C1A, JP1.9
- net N$14: now also IC1.C2B, J6.3; no longer IC1.C1B, JP1.10
- net N$15: now also IC1.D1A, J6.5; no longer IC1.C2A, JP1.11
- net N$16: now also IC1.D1B, J6.4; no longer IC1.C2B, JP1.12
- net N$17: now also IC1.D2A, J6.2; no longer IC1.D1A, JP1.13
- net N$18: now also IC1.D2B, J6.1; no longer IC1.D1B, JP1.14
- net N$2: now also IC1.A1B, J5.7; no longer IC1.A1A, JP1.1
- net N$5: now also IC1.A2B, J5.3; no longer IC1.A1B, JP1.2
- net N$6: now also IC1.B1A, J5.5; no longer IC1.A2A, JP1.3
- net N$7: now also IC1.B1B, J5.4; no longer IC1.A2B, JP1.4
- net N$8: now also IC1.B2A, J5.2; no longer IC1.B1A, JP1.5
Changed lines of the file:
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@@
 <part name="IC1" library="SamacSys_Parts" deviceset="SN65LVDT388ADBT" device=""/>
 <part name="C1" library="SparkFun-Capacitors" deviceset="CAP" device="0805" value="0.1uF"/>
-<part name="JP1" library="pinhead" library_urn="urn:adsk.eagle:library:325" deviceset="PINHD-2X8" device="/90" package3d_urn="urn:adsk.eagle:package:22488/2" value="16"/>
 <part name="IC2" library="SamacSys_Parts" deviceset="SN65LVDT388ADBT" device=""/>
 <part name="C3" library="SparkFun-Capacitors" deviceset="CAP" device="0805" value="0.1uF"/>
@@
 <attribute name="OC_NEWARK" value="unknown"/>
 </part>
+<part name="J5" library="SparkFun-Connectors" deviceset="RJ45-8" device="PTH" value="RJ45"/>
+<part name="J6" library="SparkFun-Connectors" deviceset="RJ45-8" device="PTH" value="RJ45"/>
 </parts>
 <sheets>
@@
 <attribute name="VALUE" x="120.396" y="230.759" size="1.778" layer="96" rot="R180"/>
 </instance>
-<instance part="JP1" gate="A" x="48.26" y="256.54" smashed="yes">
-<attribute name="NAME" x="41.91" y="267.335" size="1.778" layer="95"/>
-<attribute name="VALUE" x="41.91" y="241.3" size="1.778" layer="96"/>
-</instance>
 <instance part="IC2" gate="G$1" x="66.04" y="210.82" smashed="yes">
 <attribute name="NAME" x="72.39" y="218.44" size="1.778" layer="95" align="center-left"/>
@@
 <attribute name="NAME" x="52.832" y="326.136" size="1.778" layer="95" rot="R180"/>
 </instance>
+<instance part="J5" gate="JP1" x="50.8" y="266.7" smashed="yes" rot="R180">
+<attribute name="NAME" x="55.88" y="256.032" size="1.778" layer="95" rot="R180"/>
+<attribute name="VALUE" x="55.88" y="281.94" size="1.778" layer="95" rot="R180"/>
+</instance>
+<instance part="J6" gate="JP1" x="50.8" y="238.76" smashed="yes" rot="R180">
+<attribute name="NAME" x="55.88" y="228.092" size="1.778" layer="95" rot="R180"/>
+<attribute name="VALUE" x="55.88" y="254" size="1.778" layer="95" rot="R180"/>
+</instance>
 </instances>
 <busses>
@@
 </segment>
 </net>
-<net name="N$2" class="0">
-<segment>
-<pinref part="IC1" gate="G$1" pin="A1A"/>
-<pinref part="JP1" gate="A" pin="1"/>
-<wire x1="66.04" y1="276.86" x2="45.72" y2="264.16" width="0.1524" layer="91"/>
-</segment>
-</net>
-<net name="N$5" class="0">
-<segment>
-<pinref part="IC1" gate="G$1" pin="A1B"/>
-<pinref part="JP1" gate="A" pin="2"/>
-<wire x1="66.04" y1="274.32" x2="53.34" y2="264.16" width="0.1524" layer="91"/>
-</segment>
-</net>
-<net name="N$6" class="0">
-<segment>
-<pinref part="IC1" gate="G$1" pin="A2A"/>
-<pinref part="JP1" gate="A" pin="3"/>
-<wire x1="66.04" y1="271.78" x2="45.72" y2="261.62" width="0.1524" layer="91"/>
-</segment>
-</net>
-<net name="N$7" class="0">
-<segment>
-<pinref part="IC1" gate="G$1" pin="A2B"/>
-<pinref part="JP1" gate="A" pin="4"/>
-<wire x1="66.04" y1="269.24" x2="53.34" y2="261.62" width="0.1524" layer="91"/>
-</segment>
-</net>
-<net name="N$8" class="0">
-<segment>
-<pinref part="IC1" gate="G$1" pin="B1A"/>
-<pinref part="JP1" gate="A" pin="5"/>
-<wire x1="66.04" y1="264.16" x2="45.72" y2="259.08" width="0.1524" layer="91"/>
-</segment>
-</net>
-<net name="N$10" class="0">
-<segment>
-<pinref part="IC1" gate="G$1" pin="B1B"/>
-<pinref part="JP1" gate="A" pin="6"/>
-<wire x1="66.04" y1="261.62" x2="53.34" y2="259.08" width="0.1524" layer="91"/>
-</segment>
-</net>
-<net name="N$11" class="0">
-<segment>
-<pinref part="IC1" gate="G$1" pin="B2A"/>
-<pinref part="JP1" gate="A" pin="7"/>
-<wire x1="66.04" y1="259.08" x2="45.72" y2="256.54" width="0.1524" layer="91"/>
-</segment>
-</net>
-<net name="N$12" class="0">
-<segment>
-<pinref part="IC1" gate="G$1" pin="B2B"/>
-<pinref part="JP1" gate="A" pin="8"/>
-<wire x1="66.04" y1="256.54" x2="53.34" y2="256.54" width="0.1524" layer="91"/>
-</segment>
-</net>
-<net name="N$13" class="0">
-<segment>
-<pinref part="IC1" gate="G$1" pin="C1A"/>
-<pinref part="JP1" gate="A" pin="9"/>
-<wire x1="66.04" y1="251.46" x2="45.72" y2="254" width="0.1524" layer="91"/>
-</segment>
-</net>
-<net name="N$14" class="0">
-<segment>
-<pinref part="IC1" gate="G$1" pin="C1B"/>
-<pinref part="JP1" gate="A" pin="10"/>
-<wire x1="66.04" y1="248.92" x2="53.34" y2="254" width="0.1524" layer="91"/>
-</segment>
-</net>
-<net name="N$15" class="0">
-<segment>
-<pinref part="IC1" gate="G$1" pin="C2A"/>
-<pinref part="JP1" gate="A" pin="11"/>
-<wire x1="66.04" y1="246.38" x2="45.72" y2="251.46" width="0.1524" layer="91"/>
-</segment>
-</net>
-<net name="N$16" class="0">
-<segment>
-<pinref part="IC1" gate="G$1" pin="C2B"/>
-<pinref part="JP1" gate="A" pin="12"/>
-<wire x1="66.04" y1="243.84" x2="53.34" y2="251.46" width="0.1524" layer="91"/>
-</segment>
-</net>
-<net name="N$17" class="0">
-<segment>
-<pinref part="IC1" gate="G$1" pin="D1A"/>
-<pinref part="JP1" gate="A" pin="13"/>
-<wire x1="66.04" y1="238.76" x2="45.72" y2="248.92" width="0.1524" layer="91"/>
-</segment>
-</net>
-<net name="N$18" class="0">
-<segment>
-<pinref part="IC1" gate="G$1" pin="D1B"/>
-<pinref part="JP1" gate="A" pin="14"/>
-<wire x1="66.04" y1="236.22" x2="53.34" y2="248.92" width="0.1524" layer="91"/>
-</segment>
-</net>
-<net name="N$19" class="0">
-<segment>
-<pinref part="IC1" gate="G$1" pin="D2A"/>
-<pinref part="JP1" gate="A" pin="15"/>
-<wire x1="66.04" y1="233.68" x2="45.72" y2="246.38" width="0.1524" layer="91"/>
-</segment>
-</net>
-<net name="N$20" class="0">
-<segment>
-<pinref part="IC1" gate="G$1" pin="D2B"/>
-<pinref part="JP1" gate="A" pin="16"/>
-<wire x1="66.04" y1="231.14" x2="53.34" y2="246.38" width="0.1524" layer="91"/>
-</segment>
-</net>
 <net name="N$4" class="0">
 <segment>
@@
 </segment>
 </net>
+<net name="N$1" class="0">
+<segment>
+<pinref part="IC1" gate="G$1" pin="A1A"/>
+<pinref part="J5" gate="JP1" pin="8"/>
+<wire x1="66.04" y1="276.86" x2="58.42" y2="276.86" width="0.1524" layer="91"/>
+</segment>
+</net>
+<net name="N$2" class="0">
+<segment>
+<pinref part="IC1" gate="G$1" pin="A1B"/>
+<pinref part="J5" gate="JP1" pin="7"/>
+<wire x1="66.04" y1="274.32" x2="58.42" y2="274.32" width="0.1524" layer="91"/>
+</segment>
+</net>
+<net name="N$3" class="0">
+<segment>
+<pinref part="IC1" gate="G$1" pin="A2A"/>
+<pinref part="J5" gate="JP1" pin="6"/>
+<wire x1="66.04" y1="271.78" x2="58.42" y2="271.78" width="0.1524" layer="91"/>
+</segment>
+</net>
+<net name="N$5" class="0">
+<segment>
+<pinref part="IC1" gate="G$1" pin="A2B"/>
+<pinref part="J5" gate="JP1" pin="3"/>
+<wire x1="66.04" y1="269.24" x2="58.42" y2="264.16" width="0.1524" layer="91"/>
+</segment>
+</net>
+<net name="N$6" class="0">
+<segment>
+<pinref part="IC1" gate="G$1" pin="B1A"/>
+<pinref part="J5" gate="JP1" pin="5"/>
+<wire x1="66.04" y1="264.16" x2="58.42" y2="269.24" width="0.1524" layer="91"/>
+</segment>
+</net>
+<net name="N$7" class="0">
+<segment>
+<pinref part="IC1" gate="G$1" pin="B1B"/>
+<pinref part="J5" gate="JP1" pin="4"/>
+<wire x1="66.04" y1="261.62" x2="58.42" y2="266.7" width="0.1524" layer="91"/>
+</segment>
+</net>
+<net name="N$8" class="0">
+<segment>
+<pinref part="IC1" gate="G$1" pin="B2A"/>
+<pinref part="J5" gate="JP1" pin="2"/>
+<wire x1="66.04" y1="259.08" x2="58.42" y2="261.62" width="0.1524" layer="91"/>
+</segment>
+</net>
+<net name="N$10" class="0">
+<segment>
+<pinref part="IC1" gate="G$1" pin="B2B"/>
+<pinref part="J5" gate="JP1" pin="1"/>
+<wire x1="66.04" y1="256.54" x2="58.42" y2="259.08" width="0.1524" layer="91"/>
+</segment>
+</net>
+<net name="N$11" class="0">
+<segment>
+<pinref part="IC1" gate="G$1" pin="C1A"/>
+<pinref part="J6" gate="JP1" pin="8"/>
+<wire x1="66.04" y1="251.46" x2="58.42" y2="248.92" width="0.1524" layer="91"/>
+</segment>
+</net>
+<net name="N$12" class="0">
+<segment>
+<pinref part="IC1" gate="G$1" pin="C1B"/>
+<pinref part="J6" gate="JP1" pin="7"/>
+<wire x1="66.04" y1="248.92" x2="58.42" y2="246.38" width="0.1524" layer="91"/>
+</segment>
+</net>
+<net name="N$13" class="0">
+<segment>
+<pinref part="IC1" gate="G$1" pin="C2A"/>
+<pinref part="J6" gate="JP1" pin="6"/>
+<wire x1="66.04" y1="246.38" x2="58.42" y2="243.84" width="0.1524" layer="91"/>
+</segment>
+</net>
+<net name="N$14" class="0">
+<segment>
+<pinref part="IC1" gate="G$1" pin="C2B"/>
+<pinref part="J6" gate="JP1" pin="3"/>
+<wire x1="66.04" y1="243.84" x2="58.42" y2="236.22" width="0.1524" layer="91"/>
+</segment>
+</net>
+<net name="N$15" class="0">
+<segment>
+<pinref part="IC1" gate="G$1" pin="D1A"/>
+<pinref part="J6" gate="JP1" pin="5"/>
+<wire x1="66.04" y1="238.76" x2="58.42" y2="241.3" width="0.1524" layer="91"/>
+</segment>
+</net>
+<net name="N$16" class="0">
+<segment>
+<pinref part="IC1" gate="G$1" pin="D1B"/>
+<pinref part="J6" gate="JP1" pin="4"/>
+<wire x1="66.04" y1="236.22" x2="58.42" y2="238.76" width="0.1524" layer="91"/>
+</segment>
+</net>
+<net name="N$17" class="0">
+<segment>
+<pinref part="IC1" gate="G$1" pin="D2A"/>
+<pinref part="J6" gate="JP1" pin="2"/>
+<wire x1="66.04" y1="233.68" x2="58.42" y2="233.68" width="0.1524" layer="91"/>
+</segment>
+</net>
+<net name="N$18" class="0">
+<segment>
+<pinref part="IC1" gate="G$1" pin="D2B"/>
+<pinref part="J6" gate="JP1" pin="1"/>
+<wire x1="66.04" y1="231.14" x2="58.42" y2="231.14" width="0.1524" layer="91"/>
+</segment>
+</net>
